Commit message: Add lidar model and project documentation

File: urdf/my_two_wheel_robot.urdf.xacro (robot description, xacro)
@@ -170,3 +170,31 @@
 		</joint>
 	</ros2_control>
+	<!--лидар -->
+	<link name="lidar_link">
+	<visual>
+		<geometry>
+		<cylinder length="0.05" radius="0.02"/>
+		</geometry>
+		<material name="black">
+		<color rgba="0 0 0 1"/>
+		</material>
+	</visual>
+	<collision>
+		<geometry>
+		<cylinder length="0.05" radius="0.02"/>
+		</geometry>
+	</collision>
+	<inertial>
+		<mass value="0.1" />
+		<origin xyz="0 0 0"/>
+		<inertia ixx="0.001" ixy="0.0" ixz="0.0" iyy="0.001" iyz="0.0" izz="0.001" />
+	</inertial>
+	</link>
+	<!-- Фиксированный шарнир между базой и лидаром -->
+	<joint name="lidar_joint" type="fixed">
+	<parent link="base_link"/>
+	<child link="lidar_link"/>
+	<!-- Смещение (xyz) и ориентация (rpy) лидара относительно base_link -->
+	<origin xyz="0 0 0.2" rpy="0 0 0"/>
+	</joint>
 </robot>
